File: PCB/xESC_FY_r4.kicad_pcb (KiCad board)
At the start: 2 copper layers, 49.5 x 29 mm, 31 parts, among them J1 Conn_01x09_Male, J10 OM-MB W => MC BRK, J11 Conn_01x04_Pin, J3 Conn_01x05_Male, J4 Conn_01x05_Male, J6 OM-MB U => MC SA, J7 Conn_01x06_Male, J8 Conn_01x06_Pin, J9 OM-MB V => MC +24V, Q1 BSS138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

Commit message: Bootloader capable UART, high-side power switch, free-wheeling safety, current sense adjustment
Parts:
- removed C1: .1uF, Capacitor_SMD:C_0603_1608Metric
- added D3: PNE20020ER, Diode_SMD:Nexperia_CFP3_SOD-123W, F.Cu at (269.5, 118.2)
- added R10: 100, Resistor_SMD:R_0603_1608Metric, F.Cu at (270.5, 126.1)
- added R11: 2k, Resistor_SMD:R_0603_1608Metric, F.Cu at (250.3, 115.9)
- added R12: 4k7, Resistor_SMD:R_0603_1608Metric, F.Cu at (255.0, 110.9)
- added R13: 4k7, Resistor_SMD:R_0603_1608Metric, F.Cu at (256.8, 110.9)
- added R14: 4k7, Resistor_SMD:R_0603_1608Metric, F.Cu at (258.5, 110.9)
- added TP1: UART2_TX, TestPoint:TestPoint_Pad_1.5x1.5mm, F.Cu at (236.0, 115.7)
- added TP2: UART2_RX, TestPoint:TestPoint_Pad_1.5x1.5mm, F.Cu at (236.0, 118.2)
- added U2: TPS1H200A-Q1, TPS1H200AQDGNRQ1:SOP65P490X110-9N-AHMOD, F.Cu at (263.1, 121.0)
- R9: value 3mR -> 68mR; footprint Resistor_SMD:R_2512_6332Metric -> Resistor_SMD:R_1206_3216Metric_Pad1.30x1.75mm_HandSolder
- U3: value INA180A4 -> INA139NA
- moved J11 16.3 mm to (248.9, 131.2)
- moved Q3 16.0 mm to (253.2, 126.9)
- moved R7 16.0 mm to (249.3, 127.0)
- moved R8 16.0 mm to (256.6, 127.0)
- moved R9 14.1 mm to (254.5, 119.7), turned to 0 degrees
- moved D1 11.3 mm to (244.2, 126.4), turned to 90 degrees
- moved U3 11.1 mm to (254.5, 116.2), turned to 0 degrees
- moved R6 10.9 mm to (246.0, 123.2), turned to -90 degrees
- moved R5 10.6 mm to (244.2, 123.2), turned to -90 degrees
- moved D2 10.4 mm to (246.0, 126.4), turned to 90 degrees
- moved C2 10.3 mm to (254.5, 113.4), turned to 0 degrees
- moved Q1 9.34 mm to (264.6, 125.4)
- moved R1 9.34 mm to (260.6, 125.4)
- moved R2 9.34 mm to (268.1, 126.4)
- moved C5 6.22 mm to (250.3, 119.7)
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Connections:
- Q1 pad 3: /SA_HV -> /Level Shifter 1/SIGNAL_HV
- R2 pad 2: /SA_HV -> /Level Shifter 1/SIGNAL_HV
- R9 pad 1: VM -> /VMS
- U1 pad 1: /UART_RX -> /SA
- U1 pad 10: /PROTO_GPIO -> /BRK
- U1 pad 11: /LED_GN -> Net-(U1-PA4)
- U1 pad 12: /LED_RD -> Net-(U1-PA5)
- U1 pad 14: unconnected-(U1-PA7-Pad14) -> /PROTO_GPIO
- U1 pad 15: unconnected-(U1-PA8-Pad15) -> /SHUTDOWN
- U1 pad 16: unconnected-(U1-PA9/PA11-Pad16) -> /UART_TX
- U1 pad 17: /SHUTDOWN -> /UART_RX
- U1 pad 2: unconnected-(U1-PC14-Pad2) -> /LED_RD
- U1 pad 20: /UART_TX -> /VMS_DIAG_EN
- U1 pad 3: /SA -> /LED_GN
- U1 pad 7: /CUR_SENSE -> /VMS_IN
- U1 pad 8: unconnected-(U1-PA1-Pad8) -> /~{VMS_FAULT}
- U1 pad 9: /BRK -> /CUR_SENSE
- U3 pad 3: VM -> /VMS
Routing:
- net VM: track 43.6 -> 0.00 mm, vias 6 -> 4
- net /SA_HV: track 32.9 -> 2.20 mm
- net /VMS_DIAG_EN: track 0.00 -> 24.9 mm
- net Net-(U2-IN): track 0.00 -> 17.6 mm, vias 0 -> 2
- net /VMC: track 20.3 -> 2.72 mm
- net Net-(U2-~{FAULT}): track 0.00 -> 16.8 mm, vias 0 -> 2
- net Net-(U2-DIAG_EN): track 0.00 -> 16.7 mm, vias 0 -> 2
- net /VMS_IN: track 0.00 -> 16.4 mm
- net /CUR_SENSE: track 21.9 -> 5.82 mm
- net /PROTO_GPIO: track 8.99 -> 22.3 mm, vias 0 -> 1
- net /~{VMS_FAULT}: track 0.00 -> 12.1 mm
- net /BRK_HV: track 18.0 -> 7.58 mm
- net /UART_TX: track 7.97 -> 16.9 mm
- net /SA: track 9.86 -> 18.1 mm
- net /SHUTDOWN: track 11.3 -> 18.6 mm, vias 1 -> 0
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- added copper zone on B.Cu, net +5V
- added copper zone on F.Cu, net +5V
- added copper zone on F.Cu, net /BRK_HV
- added copper zone on F.Cu, net /SA_HV
- added copper zone on F.Cu, net /VMC
- added copper zone on F.Cu, net /VMS
- added copper zone on B.Cu, net VM
- added copper zone on F.Cu, net VM
