File: PCB/xESC_YF_r4.kicad_pcb (KiCad board)
At the start: 2 copper layers, 49.5 x 29 mm, 41 parts, among them J1 Conn_01x09_Male, J10 OM-MB W => MC BRK, J11 Conn_01x04_Pin, J3 Conn_01x05_Male, J4 Conn_01x05_Male, J6 OM-MB U => MC SA, J7 Conn_01x06_Male, J8 Conn_01x06_Pin, J9 OM-MB V => MC +24V, Q1 BSS138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

Commit message: UART protection
Parts:
- removed TP1: UART2_TX, TestPoint:TestPoint_Pad_1.5x1.5mm
- removed TP2: UART2_RX, TestPoint:TestPoint_Pad_1.5x1.5mm
- added J2: Conn_01x02_Pin, Connector_PinHeader_2.54mm:PinHeader_1x02_P2.54mm_Vertical, F.Cu at (236.2, 118.4)
- added JP1: UART1_TX/UART2_TX, Jumper:SolderJumper-3_P1.3mm_Bridged12_RoundedPad1.0x1.5mm_NumberLabels, F.Cu at (233.5, 123.9)
- added JP2: UART1_RX/UART2_RX, Jumper:SolderJumper-3_P1.3mm_Bridged12_RoundedPad1.0x1.5mm_NumberLabels, F.Cu at (238.7, 123.9)
- added R17: 220, Resistor_SMD:R_0603_1608Metric, F.Cu at (233.6, 127.2)
- added R18: 220, Resistor_SMD:R_0603_1608Metric, F.Cu at (238.8, 127.2)
Connections:
- J4 pad 2: /UART_TX -> Net-(J4-Pin_2)
- J4 pad 4: /UART_RX -> Net-(J4-Pin_4)
- U1 pad 11: Net-(U1-PA4) -> /UART2_TX
- U1 pad 12: Net-(U1-PA5) -> /UART2_RX
- U1 pad 16: /UART_TX -> /UART1_TX
- U1 pad 17: /UART_RX -> /UART1_RX
Routing:
- net /UART_TX: track 16.9 -> 0.00 mm
- net /UART2_TX: track 0.00 -> 15.2 mm
- net /UART_RX: track 14.1 -> 0.00 mm
- net /UART1_TX: track 0.00 -> 9.29 mm
- net Net-(U1-PA5): track 6.79 -> 0.00 mm
- net /UART2_RX: track 0.00 -> 6.65 mm
- net Net-(U1-PA4): track 6.02 -> 0.00 mm
- net /UART1_RX: track 0.00 -> 5.90 mm
- net Net-(J4-Pin_2): track 0.00 -> 3.12 mm
- net Net-(J4-Pin_4): track 0.00 -> 3.06 mm
- net /SHUTDOWN: track 18.6 -> 18.8 mm, vias 0 -> 1
- net GND: vias 7 -> 9

Commit message: Cleanup
Parts:
- R5, R6: value 1k -> 150R
Routing:
- net /UART2_RX: track 6.65 -> 12.7 mm, vias 0 -> 1
- net Net-(JP2-C): track 0.00 -> 2.38 mm
- net Net-(JP1-C): track 0.00 -> 2.33 mm
- net GND: vias 9 -> 23

Commit message: Commissioned
Parts:
- R9: value 82mR -> 75mR; footprint Resistor_SMD:R_0805_2012Metric_Pad1.20x1.40mm_HandSolder -> Resistor_SMD:R_2010_5025Metric_Pad1.40x2.65mm_HandSolder
- U1: value STM32C011F6Px -> STM32C011F6P6
- U2: value TPS1H200A-Q1 -> TPS1H200A
- moved JP2 1.53 mm to (239.0, 125.4)
- moved JP1 1.06 mm to (234.2, 123.2)
- moved R18 0.84 mm to (238.1, 127.7), turned to 0 degrees
- moved R9 0.55 mm to (254.5, 119.7)
- moved J2 0.50 mm to (236.8, 118.4)
- moved R17 0.50 mm to (233.6, 126.7)
Routing:
- net /VMS: track 11.1 -> 21.3 mm, vias 0 -> 2
- net /UART1_RX: track 5.90 -> 8.07 mm
- net /UART2_RX: track 12.7 -> 14.8 mm
- net /SHUTDOWN: track 18.8 -> 20.2 mm
- net /UART1_TX: track 9.29 -> 8.23 mm
- net /UART2_TX: track 15.2 -> 14.2 mm
- net /PROTO_GPIO: track 22.1 -> 21.3 mm
- net Net-(JP1-C): track 2.33 -> 2.94 mm
- net Net-(J4-Pin_2): track 3.12 -> 3.62 mm
- net GND: vias 23 -> 29
Other:
- board text added: "3V3"
- board text added: "5V"
- board text added: "BRK"
- board text added: "CLK"
- board text added: "DIO"
- board text added: "GND"
- board text added: "HV"
- board text added: "LV"
- board text added: "PA7"
- board text added: "RST"
- board text added: "RX"
- board text added: "SA"
- board text added: "SHUTDOWN"
- board text added: "TX"
- board text added: "VM"
- board text added: "VMC"
- board text added: "xESC_YF_r4 v1.0"
- board text added: "~{RS}"

Commit message: Fix high impedance SA input and remove proto parts
Parts:
- R1: value 1k -> 47k
- R5, R6: value 150R -> 220
Connections:
- net /Level Shifter 1/SIGNAL_HV renamed Net-(Q1-D)
Changed lines of the file:
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@@
 	(net 13 "+5V")
 	(net 14 "unconnected-(U5-NC-Pad4)")
-	(net 15 "/Level Shifter 1/SIGNAL_HV")
+	(net 15 "Net-(Q1-D)")
 	(net 16 "/VMS")
 	(net 17 "/SWDIO")
@@
 		)
 		(property ki_fp_filters "R_*")
-		(sheetname "Level Shifter 1")
-		(sheetfile "LEVEL_SHIFTER.kicad_sch")
-		(attr smd)
+		(sheetname "Stammblatt")
+		(sheetfile "xESC_YF_r4.kicad_sch")
+		(attr smd exclude_from_bom dnp)
 		(fp_line
 			(start -0.227064 -0.735)
@@
 			(layers "F.Cu" "F.Paste" "F.Mask")
 			(roundrect_rratio 0.208333)
-			(net 15 "/Level Shifter 1/SIGNAL_HV")
+			(net 15 "Net-(Q1-D)")
 			(pintype "passive")
 		)
@@
 			)
 		)
-		(property "Value" "150R"
+		(property "Value" "220"
 			(at 0 1.43 90)
 			(layer "F.Fab")
@@
 			)
 		)
-		(property "Stock_PN" "R-603-150-.1W-1%"
+		(property "Stock_PN" "R-603-220-.1W-1%"
 			(at 0 0 -90)
 			(unlocked yes)
@@
 			)
 		)
-		(property "Digikey" "311-150HRCT-ND"
+		(property "Digikey" "311-220HRCT-ND"
 			(at 0 0 -90)
 			(unlocked yes)
@@
 			)
 		)
-		(property "Part Number" "RC0603FR-07150RL"
+		(property "Part Number" "RC0603FR-07220RL"
 			(at 0 0 -90)
 			(unlocked yes)
@@
 		)
 		(property ki_fp_filters "SOT?23*")
-		(sheetname "Level Shifter 3")
-		(sheetfile "LEVEL_SHIFTER.kicad_sch")
-		(attr smd)
+		(sheetname "Stammblatt")
+		(sheetfile "xESC_YF_r4.kicad_sch")
+		(attr smd exclude_from_bom dnp)
 		(fp_line
 			(start 0 -1.56)
@@
 			(layers "F.Cu" "F.Paste" "F.Mask")
 			(roundrect_rratio 0.25)
-			(net 15 "/Level Shifter 1/SIGNAL_HV")
+			(net 15 "Net-(Q1-D)")
 			(pintype "passive")
 		)
@@
 		)
 		(property ki_fp_filters "R_*")
-		(sheetname "Level Shifter 3")
-		(sheetfile "LEVEL_SHIFTER.kicad_sch")
-		(attr smd)
+		(sheetname "Stammblatt")
+		(sheetfile "xESC_YF_r4.kicad_sch")
+		(attr smd exclude_from_bom dnp)
 		(fp_line
 			(start -0.227064 0.735)
@@
 		)
 		(property ki_fp_filters "R_*")
-		(sheetname "Level Shifter 2")
-		(sheetfile "LEVEL_SHIFTER.kicad_sch")
+		(sheetname "Stammblatt")
+		(sheetfile "xESC_YF_r4.kicad_sch")
 		(attr smd)
 		(fp_line
@@
 		)
 		(property ki_fp_filters "R_*")
-		(sheetname "Level Shifter 2")
-		(sheetfile "LEVEL_SHIFTER.kicad_sch")
+		(sheetname "Stammblatt")
+		(sheetfile "xESC_YF_r4.kicad_sch")
 		(attr smd)
 		(fp_line
@@
 		)
 		(property ki_fp_filters "R_*")
-		(sheetname "Level Shifter 3")
-		(sheetfile "LEVEL_SHIFTER.kicad_sch")
-		(attr smd)
+		(sheetname "Stammblatt")
+		(sheetfile "xESC_YF_r4.kicad_sch")
+		(attr smd exclude_from_bom dnp)
 		(fp_line
 			(start -0.227064 0.735)
@@
 			)
 		)
-		(property "Value" "150R"
+		(property "Value" "220"
 			(at 0 1.43 90)
 			(layer "F.Fab")
@@
 			)
 		)
-		(property "Stock_PN" "R-603-150-.1W-1%"
+		(property "Stock_PN" "R-603-220-.1W-1%"
 			(at 0 0 -90)
 			(unlocked yes)
@@
 			)
 		)
-		(property "Digikey" "311-150HRCT-ND"
+		(property "Digikey" "311-220HRCT-ND"
 			(at 0 0 -90)
 			(unlocked yes)
@@
 			)
 		)
-		(property "Part Number" "RC0603FR-07150RL"
+		(property "Part Number" "RC0603FR-07220RL"
 			(at 0 0 -90)
 			(unlocked yes)
@@
 			)
 		)
-		(property "Value" "1k"
+		(property "Value" "47k"
 			(at 0 1.65 90)
 			(layer "F.Fab")
@@
 			)
 		)
-		(property "Stock_PN" "R-805-1K-.125W-1%"
+		(property "Stock_PN" "R-805-47K-.125W-1%"
 			(at 0 0 -90)
 			(unlocked yes)
@@
 			)
 		)
-		(property "Digikey" "311-1.00KCRCT-ND"
+		(property "Digikey" ""
 			(at 0 0 -90)
 			(unlocked yes)
@@
 			)
 		)
-		(property "Part Number" "RC0805FR-071KL"
+		(property "Part Number" ""
 			(at 0 0 -90)
 			(unlocked yes)
@@
 			)
 		)
-		(property "LCSC" "C95781"
+		(property "LCSC" ""
 			(at 0 0 -90)
 			(unlocked yes)
@@
 		)
 		(property ki_fp_filters "R_*")
-		(sheetname "Level Shifter 1")
-		(sheetfile "LEVEL_SHIFTER.kicad_sch")
+		(sheetname "Stammblatt")
+		(sheetfile "xESC_YF_r4.kicad_sch")
 		(attr smd)
 		(fp_line
@@
 		)
 		(property ki_fp_filters "SOT?23*")
-		(sheetname "Level Shifter 2")
-		(sheetfile "LEVEL_SHIFTER.kicad_sch")
+		(sheetname "Stammblatt")
+		(sheetfile "xESC_YF_r4.kicad_sch")
 		(attr smd)
 		(fp_line
@@
 		)
 		(property ki_fp_filters "SOT?23*")
-		(sheetname "Level Shifter 1")
-		(sheetfile "LEVEL_SHIFTER.kicad_sch")
+		(sheetname "Stammblatt")
+		(sheetfile "xESC_YF_r4.kicad_sch")
 		(attr smd)
 		(fp_line
@@
 			(layers "F.Cu" "F.Paste" "F.Mask")
 			(roundrect_rratio 0.25)
-			(net 15 "/Level Shifter 1/SIGNAL_HV")
+			(net 15 "Net-(Q1-D)")
 			(pinfunction "D")
 			(pintype "passive")
