File: PCB/xESC_YF_r4.kicad_sch (KiCad schematic)
At the start: 50 parts, among them J1 Conn_01x09_Male, J10 OM-MB W => MC BRK, J2 Conn_01x03_Pin, J3 Conn_01x05_Male, J4 Conn_01x05_Male, J6 OM-MB U <= MC SA, J7 Conn_01x06_Male, J8 Conn_01x06_Pin, J9 OM-MB V => MC +24V, Q1 2N7002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

Commit message: Add next version comments
Other:
- note added: "Current-Sense and Current-Limit Calculations ---------------------- Rev4 Motor specs: I_{nom} = 30W/24V = 1.25A I_{typ_load} = 180mA (free running) to 800mA (heavy load) I_{max} = 1.5A I_{idle} = 10-12mA I_{spin-empty} = 190mA Current-Sense calc: K = 500 R_{CS} = (V_{CS} * K) / I_{OUT} = (3V * 500) / 1.5A = 1000 Ohm I_{OUT} = 1.5A => V_{CS} = 3V V_{cs,H} >= 3.13V (usable ADC range = 0-3.1V) Curre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"
- note added: "TODO ----- - Change: - D5 to: MM3Z3V3, SOD-323, i.e. C123917 - R16 to: 1k - Rcl R14 to 750 Ohm or similar with <= 1%"
- note removed: "Current-Sense and Current-Limit Calculations ---------------------- Rev4 Motor specs: I_{nom} = 30W/24V = 1.25A I_{typ_load} = 180mA (free running) to 800mA (heavy load) I_{max} = 1.5A I_{idle} = 12mA Current-Sense calc: K = 500 R_{CS} = (V_{CS} * K) / I_{OUT} = (3V * 500) / 1.5A = 1000 Ohm I_{OUT} = 1.5A => V_{CS} = 3V V_{cs,H} >= 3.13V (usable ADC range = 0-3.1V) Current-Limit calc: V_{cl,th} =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"
Changed lines of the file:
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@@
 		)
 	)
-	(text "Current-Sense and Current-Limit Calculations\n----------------------\nRev4 Motor specs:\nI_{nom} = 30W/24V = 1.25A\nI_{typ_load} = 180mA (free running) to 800mA (heavy load)\nI_{max} = 1.5A\nI_{idle} = 12mA\n\nCurrent-Sense calc:\nK = 500\nR_{CS} = (V_{CS} * K) / I_{OUT} = (3V * 500) / 1.5A = 1000 Ohm\n\nI_{OUT} = 1.5A => V_{CS} = 3V\nV_{cs,H} >= 3.13V (usable ADC range = 0-3.1V)\n\nCurrent-Limit calc:\nV_{cl,th} = 1.233\nK_{CL} = 2000\nR_{CL} = (V_{cl,th} * K_{CL}) / I_{OUT} = (1.233 * 2000) / 1.5A = 1644 Ohm\nMore common R_{CL} = 1.8k Ohm\nI_{OUT-limit} = (V_{cl,th} * K_{CL}) / R_{CL} = (1.233 * 2000) / 1800 = 1.37A\n"
+	(text "Current-Sense and Current-Limit Calculations\n----------------------\nRev4 Motor specs:\nI_{nom} = 30W/24V = 1.25A\nI_{typ_load} = 180mA (free running) to 800mA (heavy load)\nI_{max} = 1.5A\nI_{idle} = 10-12mA\nI_{spin-empty} = 190mA\n\nCurrent-Sense calc:\nK = 500\nR_{CS} = (V_{CS} * K) / I_{OUT} = (3V * 500) / 1.5A = 1000 Ohm\n\nI_{OUT} = 1.5A => V_{CS} = 3V\nV_{cs,H} >= 3.13V (usable ADC range = 0-3.1V)\n\nCurrent-Limit calc:\nV_{cl,th} = 1.233\nK_{CL} = 2000\nR_{CL} = (V_{cl,th} * K_{CL}) / I_{OUT} = (1.233 * 2000) / 1.5A = 1644 Ohm\nMore common R_{CL} = 1.8k Ohm\nI_{OUT-limit} = (V_{cl,th} * K_{CL}) / R_{CL} = (1.233 * 2000) / 1800 = 1.37A\n"
 		(exclude_from_sim no)
 		(at 297.434 85.344 0)
@@
 			)
 			(justify left)
+		)
+	)
+	(text "TODO\n-----\n- Change:\n  - D5 to: MM3Z3V3, SOD-323, i.e. C123917\n  - R16 to: 1k\n  - Rcl R14 to 750 Ohm or similar with <= 1%"
+		(exclude_from_sim no)
+		(at 199.39 19.812 0)
+		(effects
+			(font
+				(size 1.524 1.524)
+				(thickness 0.3048)
+				(bold yes)
+				(color 255 0 26 1)
+			)
+			(justify left)
