File: PCB/v1.0/xESC_YF_r4.kicad_sch (KiCad schematic)
At the start: 44 parts, among them J1 Conn_01x09_Male, J10 OM-MB W => MC BRK, J11 Conn_01x04_Pin, J2 Conn_01x02_Pin, J3 Conn_01x05_Male, J4 Conn_01x05_Male, J6 OM-MB U => MC SA, J7 Conn_01x06_Male, J8 Conn_01x06_Pin, J9 OM-MB V => MC +24V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

Commit message: Archive PCB v1.0 and start v2.0
Parts:
- removed Q1, Q2, Q3: BSS138, Package_TO_SOT_SMD:SOT-23, symbol Transistor_FET:BSS138
- removed R1, R2, R3, R4, R7, R8: 1k, Resistor_SMD:R_0805_2012Metric_Pad1.20x1.40mm_HandSolder, symbol Device:R
- R5, R6: value 220 -> 150R; Digikey 311-220HRCT-ND -> 311-150HRCT-ND; Part Number RC0603FR-07220RL -> RC0603FR-07150RL; Stock_PN R-603-220-.1W-1% -> R-603-150-.1W-1%
Connections:
- net Level Shifter 1/SIGNAL_HV: now reaches R10.1
Other:
- added sheet Level Shifter 1 (LEVEL_SHIFTER.kicad_sch)
- added sheet Level Shifter 2 (LEVEL_SHIFTER.kicad_sch)
- added sheet Level Shifter 3 (LEVEL_SHIFTER.kicad_sch)
- note removed: "Alt. 47k"
- note removed: "Alt. remove"
- note removed: "int. PullUp = Auto-Retry?"
- moved on the sheet: J10
